Commit message: edit

File: multi_robot_description/urdf/multi_world.urdf.xacro (robot description, xacro)
@@ -30,46 +30,5 @@
   <!-- end of color macros -->
   <!-- Stand macros -->
-	<link name="stand_Base1">
-    <inertial>
-      <mass value="1000" />
-      <origin xyz="0 0 0.5" rpy="0 0 0" />
-      <inertia ixx="0.01" ixy="0" ixz="0" iyy="0.01" iyz="0" izz="0.01" />
-    </inertial>
-		<visual>
-      <origin xyz="0 0 0.5" rpy="0 0 0" />
-      <geometry>
-        <cylinder radius="0.08" length="0.9"/>
-      </geometry>
-      <material name="orange_transparent"/>
-		</visual>
-		<collision>
-      <origin xyz="0 0 0.5" rpy="0 0 0" />
-      <geometry>
-        <cylinder radius="0.08" length="0.9"/>
-      </geometry>
-      <material name="blue_transparent"/>
-		</collision>
-	</link>
-	<link name="stand_Base2">
-    <inertial>
-      <mass value="1000" />
-      <origin xyz="0 0 0.5" rpy="0 0 0" />
-      <inertia ixx="0.01" ixy="0" ixz="0" iyy="0.01" iyz="0" izz="0.01" />
-    </inertial>
-		<visual>
-      <origin xyz="0 0 0.5" rpy="0 0 0" />
-      <geometry>
-        <cylinder radius="0.08" length="0.9"/>
-      </geometry>
-      <material name="orange_transparent"/>
-		</visual>
-		<collision>
-      <origin xyz="0 0 0.5" rpy="0 0 0" />
-      <geometry>
-        <cylinder radius="0.08" length="0.9"/>
-      </geometry>
-      <material name="blue_transparent"/>
-		</collision>
-	</link>
+  <xacro:include filename="$(find multi_robot_description)/urdf/stand.urdf.xacro"/>
   <!-- End of stand macros-->
   <!-- Place the stand in the world -->

File: multi_robot_description/urdf/stand.urdf.xacro (robot description, xacro)
@@ -4,6 +4,5 @@
     <static>true</static>
   </gazebo>
-  <xacro:macro name="stand" params="prefix">
-	<link name="${prefix}_stand">
+	<link name="stand_Base1">
     <inertial>
       <mass value="1000" />
@@ -26,4 +25,24 @@
 		</collision>
 	</link>
-  </xacro:macro>
+	<link name="stand_Base2">
+    <inertial>
+      <mass value="1000" />
+      <origin xyz="0 0 0.5" rpy="0 0 0" />
+      <inertia ixx="0.01" ixy="0" ixz="0" iyy="0.01" iyz="0" izz="0.01" />
+    </inertial>
+		<visual>
+      <origin xyz="0 0 0.5" rpy="0 0 0" />
+      <geometry>
+        <cylinder radius="0.08" length="0.9"/>
+      </geometry>
+      <material name="orange_transparent"/>
+		</visual>
+		<collision>
+      <origin xyz="0 0 0.5" rpy="0 0 0" />
+      <geometry>
+        <cylinder radius="0.08" length="0.9"/>
+      </geometry>
+      <material name="blue_transparent"/>
+		</collision>
+	</link>
 </robot>
